File: Kicad/RGB_strip/RGB_strip.kicad_pcb (KiCad board)
At the start: 2 copper layers, 38.2 x 27.8 mm, 18 parts, among them J1 Barrel_Jack_Switch, J2 LED, J3 Conn_01x06_Female, Q1 AO3420, Q2 AO3420, Q3 AO3420, Q4 AO3420, SW1 1TS002E-2500-2500-CT, U1 MC33275DT-3.3RKG, U2 ESP-12E

Commit message: add labels
Other:
- board text added: "12v Ch1 Ch2 Ch3 Ch4"
- board text added: "RGB Strip - ESP8266 Design by Enrique Gómez CC BY-SA 4.0 Rev.: 1.1 S/N:"
- board text removed: "RGB Strip - ESP8266 Design by Enrique Gómez CC BY-SA 4.0 Rev.: 1.0 S/N:"
